File: electrical/BioreactorPCB/POWER.sch (KiCad schematic (older format))
At the start: 8 parts, among them J13 PJ-202A, Q3 FQP47P06, Q4 TL2575HV-05IKV

Commit message: added missing electrolytic capacitors for A4988 breakouts. Preliminary layout now in place
Parts:
- Q3: footprint Package_TO_SOT_THT:TO-220-3_Horizontal_TabDown -> Package_TO_SOT_THT:TO-220-3_Vertical
- Q4: footprint Package_TO_SOT_THT:TO-220-5_P3.4x3.8mm_StaggerEven_Lead7.13mm_TabDown -> Package_TO_SOT_THT:TO-220-5_P3.4x3.7mm_StaggerEven_Lead3.8mm_Vertical
Changed lines of the file:
@@
 F 0 "Q3" V 2393 2350 50  0000 C CNN
 F 1 "FQP47P06" V 2484 2350 50  0000 C CNN
-F 2 "Package_TO_SOT_THT:TO-220-3_Horizontal_TabDown" H 2150 2350 50  0001 L BNN
+F 2 "Package_TO_SOT_THT:TO-220-3_Vertical" H 2150 2350 50  0001 L BNN
 F 3 "FQP47P06" H 2150 2350 50  0001 L BNN
 F 4 "None" H 2150 2350 50  0001 L BNN "Field4"
@@
 F 0 "Q4" H 6375 2790 50  0000 C CNN
 F 1 "TL2575HV-05IKV" H 6375 2699 50  0000 C CNN
-F 2 "Package_TO_SOT_THT:TO-220-5_P3.4x3.8mm_StaggerEven_Lead7.13mm_TabDown" H 6975 2625 50  0001 L CNN
+F 2 "Package_TO_SOT_THT:TO-220-5_P3.4x3.7mm_StaggerEven_Lead3.8mm_Vertical" H 6975 2625 50  0001 L CNN
 F 3 "http://www.ti.com/lit/gpn/tl2575hv-05" H 6975 2525 50  0001 L CNN
 F 4 "1-A Simple Step-Down Switching Voltage Regulators" H 6975 2425 50  0001 L CNN "Description"
