File: electrical/BioreactorPCB/BioreactorPCB.sch (KiCad schematic (older format))
At the start: 27 parts, among them IC1 AL5809-20P1-7, J1 61300311121, J2 61300311121, J3 OSTTC022162, J4 PJ-202A, J5 OSTTC022162, J6 OSTTC022162, J7 OSTTC042162, J8 OSTTC042162, J9 OSTTC042162, Q1 2N3905, Q2 IRF540N, Q3 FQP47P06, U1 OPT101P, U2 L293D, U3 LM329xZ

Commit message: Arduino code is validated and working on Arduino Nano Every and board layout updated to match latest.
Connections:
- wire segments 130 -> 136
- no-connect marks 31 -> 27
Other:
- note added: "D13 is connected\nto an internal LED.\nAvoid using this pin."
Changed lines of the file:
@@
 Wire Wire Line
 	2175 2025 2275 2025
-Text GLabel 7550 5500 0    50   Input ~ 0
+Text GLabel 7650 4050 1    50   Input ~ 0
 TEMP_OUT
-Wire Wire Line
-	7550 5500 7650 5500
 Text GLabel 2275 2650 2    50   Input ~ 0
 PH_OUT
@@
 	1    0    0    -1
 $EndComp
-NoConn ~ 6550 2000
-NoConn ~ 6550 2100
 NoConn ~ 6550 2300
 NoConn ~ 6550 2700
 NoConn ~ 6550 2800
 NoConn ~ 6550 2900
-NoConn ~ 8675 1975
-NoConn ~ 8675 2075
 NoConn ~ 8675 2275
 NoConn ~ 8675 2675
@@
 NoConn ~ 8650 4300
 NoConn ~ 8250 3800
-NoConn ~ 7650 4200
 NoConn ~ 7650 4300
 NoConn ~ 8650 5000
@@
 Wire Wire Line
 	5225 1550 5350 1550
+Wire Wire Line
+	7650 4200 7650 4050
+NoConn ~ 7650 5500
+Text Notes 6825 5625 0    50   ~ 0
+D13 is connected\nto an internal LED.\nAvoid using this pin.
+Wire Wire Line
+	8675 1975 8575 1975
+Wire Wire Line
+	8575 1975 8575 2075
+Wire Wire Line
+	8575 2075 8675 2075
+Wire Wire Line
+	6550 2000 6450 2000
+Wire Wire Line
+	6450 2000 6450 2100
+Wire Wire Line
+	6450 2100 6550 2100
 $EndSCHEMATC

Commit message: PCB rev 2.0 development underway
Parts:
- removed J3: OSTTC022162, digikey-footprints:Term_Block_1x2_P5.08MM, symbol dk_Terminal-Blocks-Wire-to-Board:OSTTC022162
- removed R1: 1M, Resistor_THT:R_Axial_DIN0204_L3.6mm_D1.6mm_P5.08mm_Horizontal, symbol Device:R
- removed R4: 2.2K, Resistor_THT:R_Axial_DIN0204_L3.6mm_D1.6mm_P5.08mm_Horizontal, symbol Device:R
- removed R5: 10K, Resistor_THT:R_Axial_DIN0204_L3.6mm_D1.6mm_P5.08mm_Horizontal, symbol Device:R
- removed R6: 22K, Resistor_THT:R_Axial_DIN0204_L3.6mm_D1.6mm_P5.08mm_Horizontal, symbol Device:R
- removed U1: OPT101P, digikey-footprints:DIP-8_W7.62mm, symbol dk_Optical-Sensors-Ambient-Light-IR-UV-Sensors:OPT101P
- removed U3: LM329xZ, Package_TO_SOT_THT:TO-92_Inline, symbol Reference_Voltage:LM329xZ
- added D1: LED, LED_THT:LED_D5.0mm_Horizontal_O3.81mm_Z9.0mm, symbol Device:LED
- added H1, H2, H3, H4, H5, H6, H7, H8: MountingHole_Pad, MountingHole:MountingHole_3.2mm_M3_DIN965_Pad, symbol Mechanical:MountingHole_Pad
- added IC2: VEML7700-TR, VEML7700-TR:VEML7700, symbol VEML7700-TR:VEML7700-TR
- added J10, J3: 171856-0006, 171856-0006:HDRV6W99P0X254_1X6_1509X635X1100P, symbol 171856-0006:171856-0006
- added S1: GW12RCH, GW12RCH:GW12RCH, symbol GW12RCH:GW12RCH
Connections:
- net labels added: +3V3, GND2, SCL, SDA
- net labels removed: PHOTO_OUT
- wire segments 136 -> 151
- no-connect marks 27 -> 28
Other:
- note removed: "LED connected\nto this terminal\nblock"
- moved on the sheet: J4, J8, Q3

Commit message: another intermediate
Parts:
- added C? (x2): C_Small, symbol Device:C_Small
- added C?: 100 uF, symbol Device:CP
- added C?: 330 uF, symbol Device:CP
- added C?: .1 uF, symbol Device:CP
- added C?: 22 uF, symbol Device:CP
- added C? (x2): .1 uF, symbol Device:C
- added C?: C, symbol Device:C
- added D?: 1N5819, Diode_THT:D_DO-41_SOD81_P10.16mm_Horizontal, symbol Diode:1N5819
- added IC?: TL760M33QKVURQ1, KVU-(R-PSFM-G3), symbol TL760M33QKVURQ1:TL760M33QKVURQ1
- added J?: USB_B, symbol Connector:USB_B
- added J?: Conn_02x03_Odd_Even, symbol Connector_Generic:Conn_02x03_Odd_Even
- added L?: 330 mH, symbol Device:L
- added Q?: TL2575HV-05IKV, TO170P470X1016X2338-5P, symbol TL2575HV-05IKV:TL2575HV-05IKV
- added R?: 10K, Resistor_THT:R_Axial_DIN0204_L3.6mm_D1.6mm_P5.08mm_Horizontal, symbol Device:R
- added U?: ATMEGA328-PU, digikey-footprints:DIP-28_W7.62mm, symbol dk_Embedded-Microcontrollers:ATMEGA328-PU
- added U?: FT232RL, Package_SO:SSOP-28_5.3x10.2mm_P0.65mm, symbol Interface_USB:FT232RL
- added Y?: 16 mHz, symbol Device:Crystal
Connections:
- net +3V3: now also C?.1, IC?.2 (OUTPUT)
- net +5V: now also C?.1, C?.1, C?.1, C?.2, IC?.1 (INPUT), J?.2 (Pin_2), L?.2, Q?.4 (FEEDBACK), R?.2, U?.20 (AVCC), U?.20 (VCC), U?.21 (AREF), U?.4 (VCCIO), U?.7 (VCC)
- net GND: now also C?.1, C?.1, C?.2, C?.2, C?.2, C?.2, C?.2, C?.2, D?.2 (A), IC?.3 (GND_(TAB)), J?.4 (GND), J?.5 (Shield), J?.6 (Pin_6), Q?.3 (GND), Q?.5 (~ON~/OFF), U?.18 (GND), U?.21 (GND), U?.22 (GND), U?.25 (AGND), U?.7 (GND), U?.8 (GND)
- new net: C?.1, Q?.1 (VIN)
- new net: D?.1 (K), L?.1, Q?.2 (OUTPUT)
- new net: C?.1, J?.5 (Pin_5), R?.1, U?.1 (PC6)
- new net: C?.2, U?.10 (PB7), Y?.1
- new net: C?.1, U?.9 (PB6), Y?.2
- new net: C?.2, U?.2 (DTR)
- new net MISO: J?.1 (Pin_1), U?.18 (PB4)
- new net MOSI: J?.4 (Pin_4), U?.17 (PB3)
- new net SCK: J?.3 (Pin_3), U?.19 (PB5)
- no-connect marks 28 -> 42

Commit message: Rev 2.0 schematic ready
Parts:
- removed A2: Arduino_Nano_v3.x, Module:Arduino_Nano, symbol MCU_Module:Arduino_Nano_v3.x
- removed C?: .1 uF, symbol Device:CP
- removed C?: 22 uF, symbol Device:CP
- removed IC?: TL760M33QKVURQ1, KVU-(R-PSFM-G3), symbol TL760M33QKVURQ1:TL760M33QKVURQ1
- removed U?: ATMEGA328-PU, digikey-footprints:DIP-28_W7.62mm, symbol dk_Embedded-Microcontrollers:ATMEGA328-PU
- added D2, D3: LED, symbol Device:LED
- added R1, R4: 330, symbol Device:R
- added R5, R6: R, symbol Device:R
- added U3: ATMEGA328P-AUR, digikey-footprints:TQFP-32_7x7mm, symbol dk_Embedded-Microcontrollers:ATMEGA328P-AUR
- C3: renamed from C?; value C -> .1 uF
- C4, C5: renamed from C?; value C_Small -> 22 pf
- gave numbers to parts that had none: 12
Connections:
- net +3V3: now also U1.17 (3V3OUT)
- net +5V: now also D2.2 (A), D3.2 (A), U3.18 (AVCC), U3.20 (AREF), U3.4 (VCC), U3.6 (VCC)
- net GND: now also U3.21 (GND), U3.3 (GND), U3.5 (GND)
- net MISO: now also U3.16 (PB4)
- net MOSI: now also U3.15 (PB3)
- net PH_OUT: now also U3.24 (PC1)
- net SCK: now also U3.17 (PB5)
- net SCL: now also U3.28 (PC5)
- net SDA: now also U3.27 (PC4)
- net TEMP_OUT: now also U3.25 (PC2)
- net D7: now reaches U2.1 (EN1,2)
- net D7: now also U3.11 (PD7)
- net D8: now reaches U2.2 (1A)
- net D8: now also U3.12 (PB0)
- net D9: now reaches R3.2
- net D9: now also U3.13 (PB1)
- net D2: now reaches A3.16 (DIR)
- net D2: now also U3.32 (PD2)
- net D3: now reaches A3.15 (STEP)
- net D3: now also U3.1 (PD3)
- net D4: now reaches A1.16 (DIR)
- net D4: now also U3.2 (PD4)
- net D5: now reaches A1.15 (STEP)
- net D5: now also U3.9 (PD5)
- net D6: now reaches R2.2
- net D6: now also U3.10 (PD6)
- net RESET: now reaches C3.1, J12.5 (Pin_5), R7.1
- net RESET: now also U3.29 (PC6)
- net at C5.2, Y1.1: now also U3.8 (PB7)
- net at C4.1, Y1.2: now also U3.7 (PB6)
- net at J11.2 (D-): now also U1.16 (USBD-)
- net at J11.3 (D+): now also U1.15 (USBD+)
- net RX: now reaches U1.1 (TXD)
- net RX: now also R5.2
- net at U1.22 (CBUS1): now also R4.1
- net at U1.23 (CBUS0): now also R1.2
- net TX: now reaches U1.5 (RXD)
- net TX: now also R6.2
- new net: R5.1, U3.30 (PD0)
- new net: R6.1, U3.31 (PD1)
- new net: D2.1 (K), R1.1
- new net: D3.1 (K), R4.2
- no-connect marks 42 -> 33
Other:
- note added: "TEMP_OUT is now D16"
- moved on the sheet: A1, A3, C1, C2, C3, C4, C5, C6, C7, C8, C9, D1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

Commit message: updates WIP to v 2.0
Parts:
- removed J3: 171856-0006, 171856-0006:HDRV6W99P0X254_1X6_1509X635X1100P, symbol 171856-0006:171856-0006
- added J13, J3: Conn_01x05_Male, Connector_Molex:Molex_KK-254_AE-6410-05A_1x05_P2.54mm_Vertical, symbol Connector:Conn_01x05_Male
- added S2: PEC11R-4215F-S0024, digikey-footprints:Rotary_Encoder_Switched_PEC11R, symbol dk_Encoders:PEC11R-4215F-S0024
- C1, C2: footprint Capacitor_THT:.1in_pitch -> Capacitor_THT:CP_Radial_Tantal_D5.0mm_P2.50mm
- C3, C6, C7: footprint (none) -> Capacitor_THT:CP_Radial_Tantal_D5.0mm_P2.50mm
- C4, C5: footprint (none) -> Capacitor_THT:CP_Radial_Tantal_D4.5mm_P2.50mm
- C8, C9: footprint (none) -> Capacitor_THT:CP_Radial_D5.0mm_P2.50mm
- D2, D3: footprint (none) -> LED_THT:LED_D5.0mm_Horizontal_O3.81mm_Z9.0mm
- J11: footprint (none) -> Connector_USB:USB_B_Amphenol_MUSB-D511_Vertical_Rugged
- J12: footprint (none) -> Connector_PinHeader_2.54mm:PinHeader_2x03_P2.54mm_Horizontal
- L1: value 330 mH -> 330 uH; footprint (none) -> Inductor_THT:L_Radial_D12.0mm_P6.00mm_MuRATA_1900R; Field4 (none) -> 118-6100-331K-RC-ND
- Q4: footprint TO170P470X1016X2338-5P -> Package_TO_SOT_THT:TO-220-5_P3.4x3.8mm_StaggerEven_Lead7.13mm_TabDown_Heatsink
- R1, R4: footprint (none) -> Resistor_THT:R_Axial_DIN0204_L3.6mm_D1.6mm_P5.08mm_Horizontal
- R5, R6: value R -> 1K; footprint (none) -> Resistor_THT:R_Axial_DIN0204_L3.6mm_D1.6mm_P5.08mm_Horizontal
- Y1: footprint (none) -> Crystal:Crystal_HC49-U_Vertical
Connections:
- net +3V3: now also J3.4 (Pin_4)
- net GND: now also J3.2 (Pin_2)
- net GND2: now also J13.4 (Pin_4); no longer J10.2, J10.3
- net SCL: now also J3.3 (Pin_3)
- net SDA: now also J3.5 (Pin_5)
- net at IC1.2 (OUT): now also J3.1 (Pin_1)
- net at IC2.1 (SCL): now also J13.3 (Pin_3); no longer J10.4
- net at IC2.2 (VDD): now also J13.2 (Pin_2); no longer J10.5
- net at IC2.4 (SDA): now also J13.1 (Pin_1); no longer J10.6
- net at J10.1: no longer D1.2 (A)
- new net: D1.2 (A), J13.5 (Pin_5)
Other:
- moved on the sheet: C1, C2, IC1, J10, J12, J5, Q1, R2, U2

Commit message: Completed rev 2.0 schematic for real now
Parts:
- removed A1, A3: Pololu_Breakout_A4988, Module:Pololu_Breakout-16_15.2x20.3mm, symbol Driver_Motor:Pololu_Breakout_A4988
- removed C1, C3: .1 uF, Capacitor_THT:CP_Radial_Tantal_D5.0mm_P2.50mm, symbol Device:C
- removed C2: 1 uF, Capacitor_THT:CP_Radial_Tantal_D5.0mm_P2.50mm, symbol Device:C
- removed C8: 100 uF, Capacitor_THT:CP_Radial_D5.0mm_P2.50mm, symbol Device:CP
- removed C9: 330 uF, Capacitor_THT:CP_Radial_D5.0mm_P2.50mm, symbol Device:CP
- removed D1, D2, D3: LED, LED_THT:LED_D5.0mm_Horizontal_O3.81mm_Z9.0mm, symbol Device:LED
- removed D4: 1N5819, Diode_THT:D_DO-41_SOD81_P10.16mm_Horizontal, symbol Diode:1N5819
- removed H5, H6, H7, H8: MountingHole_Pad, MountingHole:MountingHole_3.2mm_M3_DIN965_Pad, symbol Mechanical:MountingHole_Pad
- removed IC2: VEML7700-TR, VEML7700-TR:VEML7700, symbol VEML7700-TR:VEML7700-TR
- removed J10: 171856-0006, 171856-0006:HDRV6W99P0X254_1X6_1509X635X1100P, symbol 171856-0006:171856-0006
- removed J11: USB_B, Connector_USB:USB_B_Amphenol_MUSB-D511_Vertical_Rugged, symbol Connector:USB_B
- removed J13: Conn_01x05_Male, Connector_Molex:Molex_KK-254_AE-6410-05A_1x05_P2.54mm_Vertical, symbol Connector:Conn_01x05_Male
- removed J4: PJ-202A, digikey-footprints:Barrel_Jack_5.5mmODx2.1mmID_PJ-202A, symbol dk_Barrel-Power-Connectors:PJ-202A
- removed J5: OSTTC022162, digikey-footprints:Term_Block_1x2_P5.08MM, symbol dk_Terminal-Blocks-Wire-to-Board:OSTTC022162
- removed J7, J9: OSTTC042162, digikey-footprints:Term_Block_1x4_P5.08mm, symbol dk_Terminal-Blocks-Wire-to-Board:OSTTC042162
- removed L1: 330 uH, Inductor_THT:L_Radial_D12.0mm_P6.00mm_MuRATA_1900R, symbol Device:L
- removed Q3: FQP47P06, FQP47P06:TO254P1067X483X2286-3, symbol FQP47P06:FQP47P06
- removed Q4: TL2575HV-05IKV, Package_TO_SOT_THT:TO-220-5_P3.4x3.8mm_StaggerEven_Lead7.13mm_TabDown_Heatsink, symbol TL2575HV-05IKV:TL2575HV-05IKV
- removed R1, R4: 330, Resistor_THT:R_Axial_DIN0204_L3.6mm_D1.6mm_P5.08mm_Horizontal, symbol Device:R
- removed S1: GW12RCH, GW12RCH:GW12RCH, symbol GW12RCH:GW12RCH
- removed S2: PEC11R-4215F-S0024, digikey-footprints:Rotary_Encoder_Switched_PEC11R, symbol dk_Encoders:PEC11R-4215F-S0024
- removed U1: FT232RL, Package_SO:SSOP-28_5.3x10.2mm_P0.65mm, symbol Interface_USB:FT232RL
- removed U2: L293D, Package_DIP:DIP-16_W7.62mm, symbol Driver_Motor:L293D
- added J4: Conn_01x06_Male, Connector_Molex:Molex_KK-254_AE-6410-06A_1x06_P2.54mm_Vertical, symbol Connector:Conn_01x06_Male
- J12: footprint Connector_PinHeader_2.54mm:PinHeader_2x03_P2.54mm_Horizontal -> Connector_PinHeader_2.54mm:PinHeader_2x03_P2.54mm_Vertical
- Q2: footprint Package_TO_SOT_THT:TO-220-3_Vertical -> Package_TO_SOT_THT:TO-220-3_Horizontal_TabDown
Connections:
- net +3V3: now also J4.1 (Pin_1); no longer J3.4 (Pin_4)
- net +5V: now also J3.5 (Pin_5), J4.6 (Pin_6)
- net GND: now also J3.4 (Pin_4), J4.4 (Pin_4); no longer J3.2 (Pin_2)
- net SCL: now also J4.3 (Pin_3); no longer J3.3 (Pin_3)
- net SDA: now also J4.2 (Pin_2); no longer J3.5 (Pin_5)
- net at IC1.2 (OUT): now also J4.5 (Pin_5); no longer J3.1 (Pin_1)
- net BUTTON: now reaches U3.14 (PB2)
- net BUTTON: now also J3.1 (Pin_1)
- net ROT_A: now reaches U3.23 (PC0)
- net ROT_A: now also J3.2 (Pin_2)
- net ROT_B: now reaches U3.26 (PC3)
- net ROT_B: now also J3.3 (Pin_3)
- no-connect marks 33 -> 4
Other:
- note removed: "D13 is connected\nto an internal LED.\nAvoid using this pin."
- note removed: "stirrer motor"
- moved on the sheet: C4, C5, C6, C7, H1, H2, H3, H4, IC1, J1, J12, J2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

Commit message: added missing electrolytic capacitors for A4988 breakouts. Preliminary layout now in place
Parts:
- C4, C5: footprint Capacitor_THT:CP_Radial_Tantal_D4.5mm_P2.50mm -> Capacitor_THT:C_Disc_D5.0mm_W2.5mm_P2.50mm
- C6, C7: footprint Capacitor_THT:CP_Radial_Tantal_D5.0mm_P2.50mm -> Capacitor_THT:C_Disc_D5.0mm_W2.5mm_P2.50mm
- Q2: footprint Package_TO_SOT_THT:TO-220-3_Horizontal_TabDown -> Package_TO_SOT_THT:TO-220-3_Vertical
Changed lines of the file:
@@
 F 0 "Q2" H 6054 2796 50  0000 L CNN
 F 1 "IRF540N" H 6054 2705 50  0000 L CNN
-F 2 "Package_TO_SOT_THT:TO-220-3_Horizontal_TabDown" H 6100 2675 50  0001 L CIN
+F 2 "Package_TO_SOT_THT:TO-220-3_Vertical" H 6100 2675 50  0001 L CIN
 F 3 "http://www.irf.com/product-info/datasheets/data/irf540n.pdf" H 5850 2750 50  0001 L CNN
 	1    5850 2750
@@
 F 0 "C6" H 5040 4271 50  0000 L CNN
 F 1 ".1 uF" H 5040 4180 50  0000 L CNN
-F 2 "Capacitor_THT:CP_Radial_Tantal_D5.0mm_P2.50mm" H 4963 4075 50  0001 C CNN
+F 2 "Capacitor_THT:C_Disc_D5.0mm_W2.5mm_P2.50mm" H 4963 4075 50  0001 C CNN
 F 3 "~" H 4925 4225 50  0001 C CNN
 	1    4925 4225
@@
 F 0 "C7" V 5573 3825 50  0000 C CNN
 F 1 ".1 uF" V 5664 3825 50  0000 C CNN
-F 2 "Capacitor_THT:CP_Radial_Tantal_D5.0mm_P2.50mm" H 5863 3675 50  0001 C CNN
+F 2 "Capacitor_THT:C_Disc_D5.0mm_W2.5mm_P2.50mm" H 5863 3675 50  0001 C CNN
 F 3 "~" H 5825 3825 50  0001 C CNN
 	1    5825 3825
@@
 F 0 "C5" V 3875 5450 50  0000 C CNN
 F 1 "22 pf" V 3950 5450 50  0000 C CNN
-F 2 "Capacitor_THT:CP_Radial_Tantal_D4.5mm_P2.50mm" H 4075 5450 50  0001 C CNN
+F 2 "Capacitor_THT:C_Disc_D5.0mm_W2.5mm_P2.50mm" H 4075 5450 50  0001 C CNN
 F 3 "~" H 4075 5450 50  0001 C CNN
 	1    4075 5450
@@
 F 0 "C4" V 3846 5150 50  0000 C CNN
 F 1 "22 pf" V 3937 5150 50  0000 C CNN
-F 2 "Capacitor_THT:CP_Radial_Tantal_D4.5mm_P2.50mm" H 4075 5150 50  0001 C CNN
+F 2 "Capacitor_THT:C_Disc_D5.0mm_W2.5mm_P2.50mm" H 4075 5150 50  0001 C CNN
 F 3 "~" H 4075 5150 50  0001 C CNN
 	1    4075 5150

Commit message: motherboard layout complete.
Connections:
- net XTAL-: now reaches C5.2, U3.8 (PB7), Y1.1
- net XTAL+: now reaches C4.1, U3.7 (PB6), Y1.2
- net RX_TX_P: now reaches R5.1, U3.30 (PD0)
- net RX_TX_N: now reaches R6.1, U3.31 (PD1)
- net RX renamed RX_TX_+
- net TX renamed RX_TX_-
Other:
- moved on the sheet: C4, C5, R5, R6, Y1
Changed lines of the file:
@@
 	5475 5750 5475 5825
 Wire Wire Line
-	3975 5300 3975 5450
-Connection ~ 3975 5300
-Wire Wire Line
-	3975 5150 3975 5300
+	3675 5300 3675 5450
+Connection ~ 3675 5300
+Wire Wire Line
+	3675 5150 3675 5300
 NoConn ~ 5075 4550
 NoConn ~ 5075 4450
@@
 L Device:R R5
 U 1 1 620E25EE
-P 6350 4350
-F 0 "R5" V 6557 4350 50  0000 C CNN
-F 1 "1K" V 6466 4350 50  0000 C CNN
-F 2 "Resistor_THT:R_Axial_DIN0204_L3.6mm_D1.6mm_P5.08mm_Horizontal" V 6280 4350 50  0001 C CNN
-F 3 "~" H 6350 4350 50  0001 C CNN
-	1    6350 4350
-	0    -1   -1   0
-$EndComp
-Text GLabel 6500 4350 2    50   Input ~ 0
-RX
+P 6475 4350
+F 0 "R5" V 6682 4350 50  0000 C CNN
+F 1 "1K" V 6591 4350 50  0000 C CNN
+F 2 "Resistor_THT:R_Axial_DIN0204_L3.6mm_D1.6mm_P5.08mm_Horizontal" V 6405 4350 50  0001 C CNN
+F 3 "~" H 6475 4350 50  0001 C CNN
+	1    6475 4350
+	0    -1   -1   0
+$EndComp
 $Comp
 L dk_Embedded-Microcontrollers:ATMEGA328P-AUR U3
@@
 Text GLabel 6425 5150 3    50   Input ~ 0
 RESET
-Text GLabel 6500 4450 2    50   Input ~ 0
-TX
 $Comp
 L Device:R R6
 U 1 1 620E0F1A
-P 6350 4450
-F 0 "R6" V 6143 4450 50  0000 C CNN
-F 1 "1K" V 6234 4450 50  0000 C CNN
-F 2 "Resistor_THT:R_Axial_DIN0204_L3.6mm_D1.6mm_P5.08mm_Horizontal" V 6280 4450 50  0001 C CNN
-F 3 "~" H 6350 4450 50  0001 C CNN
-	1    6350 4450
+P 6475 4450
+F 0 "R6" V 6268 4450 50  0000 C CNN
+F 1 "1K" V 6359 4450 50  0000 C CNN
+F 2 "Resistor_THT:R_Axial_DIN0204_L3.6mm_D1.6mm_P5.08mm_Horizontal" V 6405 4450 50  0001 C CNN
+F 3 "~" H 6475 4450 50  0001 C CNN
+	1    6475 4450
 	0    -1   -1   0
 $EndComp
@@
 L power:GND #PWR0156
 U 1 1 61DA7998
-P 3975 5300
-F 0 "#PWR0156" H 3975 5050 50  0001 C CNN
-F 1 "GND" V 3980 5172 50  0000 R CNN
-F 2 "" H 3975 5300 50  0001 C CNN
-F 3 "" H 3975 5300 50  0001 C CNN
-	1    3975 5300
-	0    1    1    0
-$EndComp
-Connection ~ 4275 5450
-Wire Wire Line
-	4175 5450 4275 5450
-Connection ~ 4275 5150
-Wire Wire Line
-	4175 5150 4275 5150
+P 3675 5300
+F 0 "#PWR0156" H 3675 5050 50  0001 C CNN
+F 1 "GND" V 3680 5172 50  0000 R CNN
+F 2 "" H 3675 5300 50  0001 C CNN
+F 3 "" H 3675 5300 50  0001 C CNN
+	1    3675 5300
+	0    1    1    0
+$EndComp
+Connection ~ 3975 5450
+Wire Wire Line
+	3875 5450 3975 5450
+Connection ~ 3975 5150
+Wire Wire Line
+	3875 5150 3975 5150
 $Comp
 L Device:C_Small C5
 U 1 1 61D9018A
-P 4075 5450
-F 0 "C5" V 3875 5450 50  0000 C CNN
-F 1 "22 pf" V 3950 5450 50  0000 C CNN
-F 2 "Capacitor_THT:C_Disc_D5.0mm_W2.5mm_P2.50mm" H 4075 5450 50  0001 C CNN
-F 3 "~" H 4075 5450 50  0001 C CNN
-	1    4075 5450
+P 3775 5450
+F 0 "C5" V 3575 5450 50  0000 C CNN
+F 1 "22 pf" V 3650 5450 50  0000 C CNN
+F 2 "Capacitor_THT:C_Disc_D5.0mm_W2.5mm_P2.50mm" H 3775 5450 50  0001 C CNN
+F 3 "~" H 3775 5450 50  0001 C CNN
+	1    3775 5450
 	0    -1   -1   0
 $EndComp
@@
 L Device:C_Small C4
 U 1 1 61D8E602
-P 4075 5150
-F 0 "C4" V 3846 5150 50  0000 C CNN
-F 1 "22 pf" V 3937 5150 50  0000 C CNN
-F 2 "Capacitor_THT:C_Disc_D5.0mm_W2.5mm_P2.50mm" H 4075 5150 50  0001 C CNN
-F 3 "~" H 4075 5150 50  0001 C CNN
-	1    4075 5150
+P 3775 5150
+F 0 "C4" V 3546 5150 50  0000 C CNN
+F 1 "22 pf" V 3637 5150 50  0000 C CNN
+F 2 "Capacitor_THT:C_Disc_D5.0mm_W2.5mm_P2.50mm" H 3775 5150 50  0001 C CNN
+F 3 "~" H 3775 5150 50  0001 C CNN
+	1    3775 5150
 	0    1    1    0
 $EndComp
@@
 Wire Wire Line
 	4750 5450 4750 5350
-Wire Wire Line
-	4275 5450 4750 5450
-Wire Wire Line
-	4525 5150 4275 5150
 Wire Wire Line
 	4525 5250 4525 5150
@@
 L Device:Crystal Y1
 U 1 1 61D3E37A
-P 4275 5300
-F 0 "Y1" V 4321 5169 50  0000 R CNN
-F 1 "16 mHz" V 4230 5169 50  0000 R CNN
-F 2 "Crystal:Crystal_HC49-U_Vertical" H 4275 5300 50  0001 C CNN
-F 3 "~" H 4275 5300 50  0001 C CNN
-	1    4275 5300
+P 3975 5300
+F 0 "Y1" V 4021 5169 50  0000 R CNN
+F 1 "16 mHz" V 3930 5169 50  0000 R CNN
+F 2 "Crystal:Crystal_HC49-U_Vertical" H 3975 5300 50  0001 C CNN
+F 3 "~" H 3975 5300 50  0001 C CNN
+	1    3975 5300
 	0    -1   -1   0
 $EndComp
@@
 $EndSheet
 Wire Wire Line
-	6075 4350 6200 4350
-Wire Wire Line
-	6075 4450 6200 4450
+	6075 4350 6325 4350
+Wire Wire Line
+	6075 4450 6325 4450
+Text GLabel 6625 4450 2    50   Input ~ 0
+RX_TX_-
+Text GLabel 6625 4350 2    50   Input ~ 0
+RX_TX_+
+Text GLabel 4525 5150 1    50   Input ~ 0
+XTAL+
+Text GLabel 4750 5350 0    50   Input ~ 0
+XTAL-
+Wire Wire Line
+	3975 5150 4525 5150
+Wire Wire Line
+	3975 5450 4750 5450
+Text GLabel 6300 4450 3    50   Input ~ 0
+RX_TX_N
+Text GLabel 6300 4350 1    50   Input ~ 0
+RX_TX_P
 $EndSCHEMATC
