File: electrical/BioreactorPCB/BioreactorPCB.sch (KiCad schematic (older format))
At the start: 25 parts, among them IC1 AL5809-20P1-7, J1 61300311121, J12 Conn_02x03_Odd_Even, J2 61300311121, J3 Conn_01x05_Male, J4 Conn_01x06_Male, J6 OSTTC022162, J8 OSTTC042162, Q1 2N3905, Q2 IRF540N, U3 ATMEGA328P-AUR, Y1 16 mHz

Commit message: Converted all nonpolarized resistors and capacitors to SMD. USB now has differential pairs that conform to design guidelines. Lots of traces, to what end? idk.
Parts:
- C4, C5, C6, C7: footprint Capacitor_THT:C_Disc_D5.0mm_W2.5mm_P2.50mm -> Capacitor_SMD:C_0603_1608Metric_Pad1.08x0.95mm_HandSolder
- R2, R3, R5, R6, R7: footprint Resistor_THT:R_Axial_DIN0204_L3.6mm_D1.6mm_P5.08mm_Horizontal -> Resistor_SMD:R_0805_2012Metric_Pad1.20x1.40mm_HandSolder
Changed lines of the file:
@@
 F 0 "R2" V 2818 2100 50  0000 C CNN
 F 1 "1K" V 2909 2100 50  0000 C CNN
-F 2 "Resistor_THT:R_Axial_DIN0204_L3.6mm_D1.6mm_P5.08mm_Horizontal" V 2955 2100 50  0001 C CNN
+F 2 "Resistor_SMD:R_0805_2012Metric_Pad1.20x1.40mm_HandSolder" V 2955 2100 50  0001 C CNN
 F 3 "~" H 3025 2100 50  0001 C CNN
 	1    3025 2100
@@
 F 0 "R3" V 5218 2750 50  0000 C CNN
 F 1 "10K" V 5309 2750 50  0000 C CNN
-F 2 "Resistor_THT:R_Axial_DIN0204_L3.6mm_D1.6mm_P5.08mm_Horizontal" V 5355 2750 50  0001 C CNN
+F 2 "Resistor_SMD:R_0805_2012Metric_Pad1.20x1.40mm_HandSolder" V 5355 2750 50  0001 C CNN
 F 3 "~" H 5425 2750 50  0001 C CNN
 	1    5425 2750
@@
 F 0 "R5" V 6682 4350 50  0000 C CNN
 F 1 "1K" V 6591 4350 50  0000 C CNN
-F 2 "Resistor_THT:R_Axial_DIN0204_L3.6mm_D1.6mm_P5.08mm_Horizontal" V 6405 4350 50  0001 C CNN
+F 2 "Resistor_SMD:R_0805_2012Metric_Pad1.20x1.40mm_HandSolder" V 6405 4350 50  0001 C CNN
 F 3 "~" H 6475 4350 50  0001 C CNN
 	1    6475 4350
@@
 F 0 "R6" V 6268 4450 50  0000 C CNN
 F 1 "1K" V 6359 4450 50  0000 C CNN
-F 2 "Resistor_THT:R_Axial_DIN0204_L3.6mm_D1.6mm_P5.08mm_Horizontal" V 6405 4450 50  0001 C CNN
+F 2 "Resistor_SMD:R_0805_2012Metric_Pad1.20x1.40mm_HandSolder" V 6405 4450 50  0001 C CNN
 F 3 "~" H 6475 4450 50  0001 C CNN
 	1    6475 4450
@@
 F 0 "C6" H 5040 4271 50  0000 L CNN
 F 1 ".1 uF" H 5040 4180 50  0000 L CNN
-F 2 "Capacitor_THT:C_Disc_D5.0mm_W2.5mm_P2.50mm" H 4963 4075 50  0001 C CNN
+F 2 "Capacitor_SMD:C_0603_1608Metric_Pad1.08x0.95mm_HandSolder" H 4963 4075 50  0001 C CNN
 F 3 "~" H 4925 4225 50  0001 C CNN
 	1    4925 4225
@@
 F 0 "C7" V 5573 3825 50  0000 C CNN
 F 1 ".1 uF" V 5664 3825 50  0000 C CNN
-F 2 "Capacitor_THT:C_Disc_D5.0mm_W2.5mm_P2.50mm" H 5863 3675 50  0001 C CNN
+F 2 "Capacitor_SMD:C_0603_1608Metric_Pad1.08x0.95mm_HandSolder" H 5863 3675 50  0001 C CNN
 F 3 "~" H 5825 3825 50  0001 C CNN
 	1    5825 3825
@@
 F 0 "R7" V 6493 5150 50  0000 C CNN
 F 1 "10K" V 6584 5150 50  0000 C CNN
-F 2 "Resistor_THT:R_Axial_DIN0204_L3.6mm_D1.6mm_P5.08mm_Horizontal" V 6630 5150 50  0001 C CNN
+F 2 "Resistor_SMD:R_0805_2012Metric_Pad1.20x1.40mm_HandSolder" V 6630 5150 50  0001 C CNN
 F 3 "~" H 6700 5150 50  0001 C CNN
 	1    6700 5150
@@
 F 0 "C5" V 3575 5450 50  0000 C CNN
 F 1 "22 pf" V 3650 5450 50  0000 C CNN
-F 2 "Capacitor_THT:C_Disc_D5.0mm_W2.5mm_P2.50mm" H 3775 5450 50  0001 C CNN
+F 2 "Capacitor_SMD:C_0603_1608Metric_Pad1.08x0.95mm_HandSolder" H 3775 5450 50  0001 C CNN
 F 3 "~" H 3775 5450 50  0001 C CNN
 	1    3775 5450
@@
 F 0 "C4" V 3546 5150 50  0000 C CNN
 F 1 "22 pf" V 3637 5150 50  0000 C CNN
-F 2 "Capacitor_THT:C_Disc_D5.0mm_W2.5mm_P2.50mm" H 3775 5150 50  0001 C CNN
+F 2 "Capacitor_SMD:C_0603_1608Metric_Pad1.08x0.95mm_HandSolder" H 3775 5150 50  0001 C CNN
 F 3 "~" H 3775 5150 50  0001 C CNN
 	1    3775 5150
