File: electrical/BioreactorPCB/BUTTON.sch (KiCad schematic (older format))
At the start: 9 parts, among them J14 Conn_01x05_Male

Commit message: Converted all nonpolarized resistors and capacitors to SMD. USB now has differential pairs that conform to design guidelines. Lots of traces, to what end? idk.
Parts:
- R10, R11, R9: footprint Resistor_THT:R_Axial_DIN0204_L3.6mm_D1.6mm_P5.08mm_Horizontal -> Resistor_SMD:R_0805_2012Metric_Pad1.20x1.40mm_HandSolder
Changed lines of the file:
@@
 F 0 "R11" V 6432 2900 50  0000 C CNN
 F 1 "10K" V 6341 2900 50  0000 C CNN
-F 2 "Resistor_THT:R_Axial_DIN0204_L3.6mm_D1.6mm_P5.08mm_Horizontal" V 6155 2900 50  0001 C CNN
+F 2 "Resistor_SMD:R_0805_2012Metric_Pad1.20x1.40mm_HandSolder" V 6155 2900 50  0001 C CNN
 F 3 "~" H 6225 2900 50  0001 C CNN
 	1    6225 2900
@@
 F 0 "R9" V 5032 2850 50  0000 C CNN
 F 1 "10K" V 4941 2850 50  0000 C CNN
-F 2 "Resistor_THT:R_Axial_DIN0204_L3.6mm_D1.6mm_P5.08mm_Horizontal" V 4755 2850 50  0001 C CNN
+F 2 "Resistor_SMD:R_0805_2012Metric_Pad1.20x1.40mm_HandSolder" V 4755 2850 50  0001 C CNN
 F 3 "~" H 4825 2850 50  0001 C CNN
 	1    4825 2850
@@
 F 0 "R10" V 4957 3350 50  0000 C CNN
 F 1 "10K" V 4866 3350 50  0000 C CNN
-F 2 "Resistor_THT:R_Axial_DIN0204_L3.6mm_D1.6mm_P5.08mm_Horizontal" V 4680 3350 50  0001 C CNN
+F 2 "Resistor_SMD:R_0805_2012Metric_Pad1.20x1.40mm_HandSolder" V 4680 3350 50  0001 C CNN
 F 3 "~" H 4750 3350 50  0001 C CNN
 	1    4750 3350
