File: electrical/BioreactorPCB/POWER.kicad_sch (KiCad schematic)
At the start: 8 parts, among them J13 PJ-202A, Q3 FQP47P06, Q4 TL2575HV-05IKV

Commit message: NOW a 4-layer pCB with drastically improved routing
Parts:
- L1: footprint Inductor_THT:L_Radial_D12.0mm_P6.00mm_MuRATA_1900R -> Inductor_SMD:L_Bourns_SRR1210A; Field4 118-6100-331K-RC-ND -> SRR1210-331MCT-ND
Changed lines of the file:
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@@
     (property "Reference" "L1" (id 0) (at 137.16 44.704 90))
     (property "Value" "330 uH" (id 1) (at 137.16 47.0154 90))
-    (property "Footprint" "Inductor_THT:L_Radial_D12.0mm_P6.00mm_MuRATA_1900R" (id 2) (at 137.16 49.53 0)
+    (property "Footprint" "Inductor_SMD:L_Bourns_SRR1210A" (id 2) (at 137.16 49.53 0)
       (effects (font (size 1.27 1.27)) hide)
     )
@@
       (effects (font (size 1.27 1.27)) hide)
     )
-    (property "Field4" "118-6100-331K-RC-ND" (id 4) (at 137.16 49.53 90)
+    (property "Field4" "SRR1210-331MCT-ND" (id 4) (at 137.16 49.53 90)
       (effects (font (size 1.27 1.27)) hide)
     )
